File: keycultTKL.kicad_sch (KiCad schematic)
At the start: 213 parts, among them J1 Conn_01x04, U1 XC6206PxxxMR, U2 W25Q128JVS, U3 RP2040, U4 SRV05-4, Y1 ABM8-272-T3

Commit message: V1.4
Parts:
- D90, D91, D92: footprint hjcustom:E6CC1206CWAY1UDA -> hjcustom:KT-0805W
Changed lines of the file:
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@@
 			)
 		)
-		(property "Footprint" "hjcustom:E6CC1206CWAY1UDA"
+		(property "Footprint" "hjcustom:KT-0805W"
 			(at 171.45 160.02 0)
 			(effects
@@
 			)
 		)
-		(property "Footprint" "hjcustom:E6CC1206CWAY1UDA"
+		(property "Footprint" "hjcustom:KT-0805W"
 			(at 168.91 102.87 0)
 			(effects
@@
 			)
 		)
-		(property "Footprint" "hjcustom:E6CC1206CWAY1UDA"
+		(property "Footprint" "hjcustom:KT-0805W"
 			(at 173.99 102.87 0)
 			(effects

Commit message: V1.4
Parts:
- R1, R2: footprint hjcustom:C_0402_1005Metric -> Capacitor_SMD:C_0603_1608Metric
- R5, R7, R8: value 100R -> 300R
Changed lines of the file:
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@@
 			)
 		)
-		(property "Footprint" "hjcustom:C_0402_1005Metric"
+		(property "Footprint" "Capacitor_SMD:C_0603_1608Metric"
 			(at 156.21 80.01 0)
 			(effects
@@
 			)
 		)
-		(property "Footprint" "hjcustom:C_0402_1005Metric"
+		(property "Footprint" "Capacitor_SMD:C_0603_1608Metric"
 			(at 156.21 77.47 0)
 			(effects
@@
 			)
 		)
-		(property "Value" "100R"
+		(property "Value" "300R"
 			(at 179.832 96.52 90)
 			(effects
@@
 			)
 		)
-		(property "Value" "100R"
+		(property "Value" "300R"
 			(at 166.116 96.52 90)
 			(effects
@@
 			)
 		)
-		(property "Value" "100R"
+		(property "Value" "300R"
 			(at 168.656 153.67 90)
 			(effects

Commit message: V1.6
Parts:
- D1, D10, D11, D12, D13, D14, D15, D16, D17, D18, D19, D2, D20, D21, D22, D23, D24, D25, D26, D27, D28, D29, D3, D30, D31, D32, D33, D34, D35, D36, D37, D38, D39, D4, D40, D41, D42, D43, D44, D45, D46, D47, D48, D49, D5, D50, D51, D52, D53, D54, D55, D56, D57, D58, D59, D6, D60, D61, D62, D63, D64, D65, D66, D67, D68, D69, D7, D70, D71, D72, D73, D74, D75, D76, D77, D78, D79, D8, D80, D81, D82, D83, D84, D85, D86, D87, D88, D89, D9: footprint ScottoKeebs_Components:Diode_SOD-123_noref -> ScottoKeebs_Components:Diode_SOD-123_noref2
- U2: footprint Package_SO:SOIC-8_5.23x5.23mm_P1.27mm -> hjcustom:SOIC-8_5.23x5.23mm_P1.27mm
- Y1: footprint Oscillator:Oscillator_SMD_EuroQuartz_XO32-4Pin_3.2x2.5mm -> hjcustom:Oscillator_SMD_EuroQuartz_XO32-4Pin_3.2x2.5mm
